File: Hardware/Amp2.sch (KiCad schematic (older format))
At the start: 23 parts

Commit message: Add second detection chain
Parts:
- removed C?: 4.7pF, CAPC1608, symbol C
- removed C? (x2): 0.1uF, CAPC1608, symbol C
- removed C? (x3): 100pF, CAPC1608, symbol C
- removed C? (x4): 0.01uF, CAPC1608, symbol C
- removed R?: 10M, RESC1608, symbol R
- removed R? (x3): 1k, RESC1608, symbol R
- removed R? (x3): 10k, RESC1608, symbol R
- removed TP?: Out1, symbol TP
- removed TP?: In1, symbol TP
- removed U? (x4): MAX4477, symbol OPAMP-DUAL
- added C?: 4.7pF, CAPC1608, symbol C
- added C? (x2): 0.1uF, CAPC1608, symbol C
- added C? (x3): 100pF, CAPC1608, symbol C
- added C? (x4): 0.01uF, CAPC1608, symbol C
- added R?: 10M, RESC1608, symbol R
- added R? (x3): 1k, RESC1608, symbol R
- added R? (x3): 10k, RESC1608, symbol R
- added TP?: Out1, symbol TP
- added TP?: In1, symbol TP
- added U? (x4): MAX4477, symbol OPAMP-DUAL
Changed lines of the file:
@@
 $Descr A4 11693 8268
 encoding utf-8
-Sheet 3 7
+Sheet 6 7
 Title "Solid State Cosmic Ray Detector"
 Date "24 sep 2013"
@@
 $Comp
 L OPAMP-DUAL U?
-U 1 1 523CFEC7
+U 1 1 52414EC5
 P 2400 3700
 F 0 "U?" H 2150 3800 50  0000 L CNN
@@
 $Comp
 L GND #PWR?
-U 1 1 523CFED3
+U 1 1 52414ECB
 P 2400 4200
 F 0 "#PWR?" H 2400 4200 30  0001 C CNN
@@
 $Comp
 L GND #PWR?
-U 1 1 523CFED9
+U 1 1 52414ED1
 P 1800 4000
 F 0 "#PWR?" H 1800 4000 30  0001 C CNN
@@
 $Comp
 L GND #PWR?
-U 1 1 523CFEDF
+U 1 1 52414ED7
 P 4300 4200
 F 0 "#PWR?" H 4300 4200 30  0001 C CNN
@@
 $Comp
 L R R?
-U 1 1 523CFEE7
+U 1 1 52414EE2
 P 1950 3000
 F 0 "R?" H 1950 3100 50  0000 C CNN
@@
 $Comp
 L C C?
-U 1 1 523CFEEF
+U 1 1 52414EED
 P 1950 2600
 F 0 "C?" H 2000 2750 60  0000 L CNN
@@
 $Comp
 L +5V #PWR?
-U 1 1 523CFEF5
+U 1 1 52414EF3
 P 2400 2500
 F 0 "#PWR?" H 2400 2590 20  0001 C CNN
@@
 $Comp
 L C C?
-U 1 1 523CFEFD
+U 1 1 52414EFE
 P 2750 2600
 F 0 "C?" H 2800 2750 60  0000 L CNN
@@
 $Comp
 L R R?
-U 1 1 523CFF0D
+U 1 1 52414F09
 P 3950 3700
 F 0 "R?" H 3950 3800 50  0000 C CNN
@@
 $Comp
 L R R?
-U 1 1 523CFF15
+U 1 1 52414F14
 P 4850 3300
 F 0 "R?" H 4850 3400 50  0000 C CNN
@@
 $Comp
 L C C?
-U 1 1 523CFF1D
+U 1 1 52414F1F
 P 4850 2900
 F 0 "C?" H 4900 3050 60  0000 L CNN
@@
 $Comp
 L GND #PWR?
-U 1 1 523CFF43
+U 1 1 52414F45
 P 3100 2600
 F 0 "#PWR?" H 3100 2600 30  0001 C CNN
@@
 $Comp
 L C C?
-U 1 1 523CFF56
+U 1 1 52414F53
 P 1250 3500
 F 0 "C?" H 1300 3650 60  0000 L CNN
@@
 $Comp
 L GND #PWR?
-U 1 1 523CFF91
+U 1 1 52414F68
 P 8300 3000
 F 0 "#PWR?" H 8300 3000 30  0001 C CNN
@@
 $Comp
 L +5V #PWR?
-U 1 1 523CFF98
+U 1 1 52414F6F
 P 7600 2900
 F 0 "#PWR?" H 7600 2990 20  0001 C CNN
@@
 $Comp
 L GND #PWR?
-U 1 1 523CFFD6
+U 1 1 52414F87
 P 9500 4600
 F 0 "#PWR?" H 9500 4600 30  0001 C CNN
@@
 $Comp
 L GND #PWR?
-U 1 1 523CFFDC
+U 1 1 52414F8D
 P 7600 4600
 F 0 "#PWR?" H 7600 4600 30  0001 C CNN
@@
 $Comp
 L GND #PWR?
-U 1 1 523CFFE2
+U 1 1 52414F93
 P 7000 4400
 F 0 "#PWR?" H 7000 4400 30  0001 C CNN
@@
 $Comp
 L TP TP?
-U 1 1 523CFFF1
+U 1 1 52414FA0
 P 10700 3600
 F 0 "TP?" H 10700 3950 60  0000 C CNN
@@
 $Comp
 L TP TP?
-U 1 1 523CFFF8
+U 1 1 52414FA7
 P 900 3400
 F 0 "TP?" H 900 3750 60  0000 C CNN
@@
 $Comp
 L OPAMP-DUAL U?
-U 2 1 523FC6E8
+U 2 1 52414FB4
 P 4900 3900
 F 0 "U?" H 4650 4000 50  0000 L CNN
@@
 $Comp
 L OPAMP-DUAL U?
-U 1 1 523FC6F1
+U 1 1 52414FBD
 P 7600 4100
 F 0 "U?" H 7350 4200 50  0000 L CNN
@@
 $Comp
 L OPAMP-DUAL U?
-U 2 1 523FC6FA
+U 2 1 52414FC6
 P 10100 4300
 F 0 "U?" H 9850 4400 50  0000 L CNN
@@
 $Comp
 L C C?
-U 1 1 524124C8
+U 1 1 52414FD1
 P 3350 3700
 F 0 "C?" H 3400 3850 60  0000 L CNN
@@
 $Comp
 L C C?
-U 1 1 524124D3
+U 1 1 52414FDC
 P 5850 3900
 F 0 "C?" H 5900 4050 60  0000 L CNN
@@
 $Comp
 L C C?
-U 1 1 524124DE
+U 1 1 52414FE7
 P 8550 4100
 F 0 "C?" H 8600 4250 60  0000 L CNN
@@
 $Comp
 L C C?
-U 1 1 5241258A
+U 1 1 52414FF2
 P 7150 3000
 F 0 "C?" H 7200 3150 60  0000 L CNN
@@
 $Comp
 L C C?
-U 1 1 52412595
+U 1 1 52414FFD
 P 10050 3300
 F 0 "C?" H 10100 3450 60  0000 L CNN
@@
 $Comp
 L R R?
-U 1 1 5241267F
+U 1 1 52415008
 P 6450 3900
 F 0 "R?" H 6450 4000 50  0000 C CNN
@@
 $Comp
 L R R?
-U 1 1 5241268A
+U 1 1 52415013
 P 9150 4100
 F 0 "R?" H 9150 4200 50  0000 C CNN
@@
 $Comp
 L R R?
-U 1 1 52412715
+U 1 1 5241501E
 P 7150 3400
 F 0 "R?" H 7150 3500 50  0000 C CNN
@@
 $Comp
 L R R?
-U 1 1 52412720
+U 1 1 52415029
 P 10050 3700
 F 0 "R?" H 10050 3800 50  0000 C CNN
@@
 $Comp
 L C C?
-U 1 1 52412801
+U 1 1 52415034
 P 7950 3000
 F 0 "C?" H 8000 3150 60  0000 L CNN

Commit message: Initial annotation
Parts:
- gave numbers to parts that had none: 21
Changed lines of the file:
@@
 $EndDescr
 $Comp
-L OPAMP-DUAL U?
+L OPAMP-DUAL U6
 U 1 1 52414EC5
 P 2400 3700
-F 0 "U?" H 2150 3800 50  0000 L CNN
+F 0 "U6" H 2150 3800 50  0000 L CNN
 F 1 "MAX4477" H 2150 3700 50  0000 L CNN
 F 2 "" H 2400 3700 60  0000 C CNN
@@
 $EndComp
 $Comp
-L GND #PWR?
+L GND #PWR51
 U 1 1 52414ECB
 P 2400 4200
-F 0 "#PWR?" H 2400 4200 30  0001 C CNN
+F 0 "#PWR51" H 2400 4200 30  0001 C CNN
 F 1 "GND" H 2400 4130 30  0001 C CNN
 F 2 "" H 2400 4200 60  0000 C CNN
@@
 $EndComp
 $Comp
-L GND #PWR?
+L GND #PWR50
 U 1 1 52414ED1
 P 1800 4000
-F 0 "#PWR?" H 1800 4000 30  0001 C CNN
+F 0 "#PWR50" H 1800 4000 30  0001 C CNN
 F 1 "GND" H 1800 3930 30  0001 C CNN
 F 2 "" H 1800 4000 60  0000 C CNN
@@
 $EndComp
 $Comp
-L GND #PWR?
+L GND #PWR52
 U 1 1 52414ED7
 P 4300 4200
-F 0 "#PWR?" H 4300 4200 30  0001 C CNN
+F 0 "#PWR52" H 4300 4200 30  0001 C CNN
 F 1 "GND" H 4300 4130 30  0001 C CNN
 F 2 "" H 4300 4200 60  0000 C CNN
@@
 $EndComp
 $Comp
-L R R?
+L R R16
 U 1 1 52414EE2
 P 1950 3000
-F 0 "R?" H 1950 3100 50  0000 C CNN
+F 0 "R16" H 1950 3100 50  0000 C CNN
 F 1 "10M" H 1950 3000 50  0000 C CNN
 F 2 "RESC1608" H 1950 3000 60  0001 C CNN
@@
 $EndComp
 $Comp
-L C C?
+L C C21
 U 1 1 52414EED
 P 1950 2600
-F 0 "C?" H 2000 2750 60  0000 L CNN
+F 0 "C21" H 2000 2750 60  0000 L CNN
 F 1 "4.7pF" H 2000 2450 60  0000 L CNN
 F 2 "CAPC1608" H 1950 2600 60  0001 C CNN
@@
 $EndComp
 $Comp
-L +5V #PWR?
+L +5V #PWR46
 U 1 1 52414EF3
 P 2400 2500
-F 0 "#PWR?" H 2400 2590 20  0001 C CNN
+F 0 "#PWR46" H 2400 2590 20  0001 C CNN
 F 1 "+5V" H 2400 2590 30  0000 C CNN
 F 2 "" H 2400 2500 60  0000 C CNN
@@
 $EndComp
 $Comp
-L C C?
+L C C22
 U 1 1 52414EFE
 P 2750 2600
-F 0 "C?" H 2800 2750 60  0000 L CNN
+F 0 "C22" H 2800 2750 60  0000 L CNN
 F 1 "0.1uF" H 2800 2450 60  0000 L CNN
 F 2 "CAPC1608" H 2750 2600 60  0001 C CNN
@@
 $EndComp
 $Comp
-L R R?
+L R R19
 U 1 1 52414F09
 P 3950 3700
-F 0 "R?" H 3950 3800 50  0000 C CNN
+F 0 "R19" H 3950 3800 50  0000 C CNN
 F 1 "1k" H 3950 3700 50  0000 C CNN
 F 2 "RESC1608" H 3950 3700 60  0001 C CNN
@@
 $EndComp
 $Comp
-L R R?
+L R R17
 U 1 1 52414F14
 P 4850 3300
-F 0 "R?" H 4850 3400 50  0000 C CNN
+F 0 "R17" H 4850 3400 50  0000 C CNN
 F 1 "10k" H 4850 3300 50  0000 C CNN
 F 2 "RESC1608" H 4850 3300 60  0001 C CNN
@@
 $EndComp
 $Comp
-L C C?
+L C C23
 U 1 1 52414F1F
 P 4850 2900
-F 0 "C?" H 4900 3050 60  0000 L CNN
+F 0 "C23" H 4900 3050 60  0000 L CNN
 F 1 "100pF" H 4900 2750 60  0000 L CNN
 F 2 "CAPC1608" H 4850 2900 60  0001 C CNN
@@
 Connection ~ 1600 3000
 $Comp
-L GND #PWR?
+L GND #PWR47
 U 1 1 52414F45
 P 3100 2600
-F 0 "#PWR?" H 3100 2600 30  0001 C CNN
+F 0 "#PWR47" H 3100 2600 30  0001 C CNN
 F 1 "GND" H 3100 2530 30  0001 C CNN
 F 2 "" H 3100 2600 60  0000 C CNN
@@
 Connection ~ 2400 2600
 $Comp
-L C C?
+L C C27
 U 1 1 52414F53
 P 1250 3500
-F 0 "C?" H 1300 3650 60  0000 L CNN
+F 0 "C27" H 1300 3650 60  0000 L CNN
 F 1 "0.01uF" H 1300 3350 60  0000 L CNN
 F 2 "CAPC1608" H 1250 3500 60  0001 C CNN
@@
 Connection ~ 7500 3400
 $Comp
-L GND #PWR?
+L GND #PWR49
 U 1 1 52414F68
 P 8300 3000
-F 0 "#PWR?" H 8300 3000 30  0001 C CNN
+F 0 "#PWR49" H 8300 3000 30  0001 C CNN
 F 1 "GND" H 8300 2930 30  0001 C CNN
 F 2 "" H 8300 3000 60  0000 C CNN
@@
 	8300 3000 8200 3000
 $Comp
-L +5V #PWR?
+L +5V #PWR48
 U 1 1 52414F6F
 P 7600 2900
-F 0 "#PWR?" H 7600 2990 20  0001 C CNN
+F 0 "#PWR48" H 7600 2990 20  0001 C CNN
 F 1 "+5V" H 7600 2990 30  0000 C CNN
 F 2 "" H 7600 2900 60  0000 C CNN
@@
 Connection ~ 10400 3700
 $Comp
-L GND #PWR?
+L GND #PWR55
 U 1 1 52414F87
 P 9500 4600
-F 0 "#PWR?" H 9500 4600 30  0001 C CNN
+F 0 "#PWR55" H 9500 4600 30  0001 C CNN
 F 1 "GND" H 9500 4530 30  0001 C CNN
 F 2 "" H 9500 4600 60  0000 C CNN
@@
 $EndComp
 $Comp
-L GND #PWR?
+L GND #PWR54
 U 1 1 52414F8D
 P 7600 4600
-F 0 "#PWR?" H 7600 4600 30  0001 C CNN
+F 0 "#PWR54" H 7600 4600 30  0001 C CNN
 F 1 "GND" H 7600 4530 30  0001 C CNN
 F 2 "" H 7600 4600 60  0000 C CNN
@@
 $EndComp
 $Comp
-L GND #PWR?
+L GND #PWR53
 U 1 1 52414F93
 P 7000 4400
-F 0 "#PWR?" H 7000 4400 30  0001 C CNN
+F 0 "#PWR53" H 7000 4400 30  0001 C CNN
 F 1 "GND" H 7000 4330 30  0001 C CNN
 F 2 "" H 7000 4400 60  0000 C CNN
@@
 Connection ~ 10700 4300
 $Comp
-L TP TP?
+L TP TP4
 U 1 1 52414FA0
 P 10700 3600
-F 0 "TP?" H 10700 3950 60  0000 C CNN
+F 0 "TP4" H 10700 3950 60  0000 C CNN
 F 1 "Out1" H 10700 3850 60  0000 C CNN
 F 2 "" H 10700 3600 60  0000 C CNN
@@
 Connection ~ 10700 3700
 $Comp
-L TP TP?
+L TP TP3
 U 1 1 52414FA7
 P 900 3400
-F 0 "TP?" H 900 3750 60  0000 C CNN
+F 0 "TP3" H 900 3750 60  0000 C CNN
 F 1 "In1" H 900 3650 60  0000 C CNN
 F 2 "" H 900 3400 60  0000 C CNN
@@
 In
 $Comp
-L OPAMP-DUAL U?
+L OPAMP-DUAL U6
 U 2 1 52414FB4
 P 4900 3900
-F 0 "U?" H 4650 4000 50  0000 L CNN
+F 0 "U6" H 4650 4000 50  0000 L CNN
 F 1 "MAX4477" H 4650 3900 50  0000 L CNN
 F 2 "" H 4900 3900 60  0000 C CNN
@@
 $EndComp
 $Comp
-L OPAMP-DUAL U?
+L OPAMP-DUAL U7
 U 1 1 52414FBD
 P 7600 4100
-F 0 "U?" H 7350 4200 50  0000 L CNN
+F 0 "U7" H 7350 4200 50  0000 L CNN
 F 1 "MAX4477" H 7350 4100 50  0000 L CNN
 F 2 "" H 7600 4100 60  0000 C CNN
@@
 $EndComp
 $Comp
-L OPAMP-DUAL U?
+L OPAMP-DUAL U7
 U 2 1 52414FC6
 P 10100 4300
-F 0 "U?" H 9850 4400 50  0000 L CNN
+F 0 "U7" H 9850 4400 50  0000 L CNN
 F 1 "MAX4477" H 9850 4300 50  0000 L CNN
 F 2 "" H 10100 4300 60  0000 C CNN
@@
 $EndComp
 $Comp
-L C C?
+L C C28
 U 1 1 52414FD1
 P 3350 3700
-F 0 "C?" H 3400 3850 60  0000 L CNN
+F 0 "C28" H 3400 3850 60  0000 L CNN
 F 1 "0.01uF" H 3400 3550 60  0000 L CNN
 F 2 "CAPC1608" H 3350 3700 60  0001 C CNN
@@
 $EndComp
 $Comp
-L C C?
+L C C29
 U 1 1 52414FDC
 P 5850 3900
-F 0 "C?" H 5900 4050 60  0000 L CNN
+F 0 "C29" H 5900 4050 60  0000 L CNN
 F 1 "0.01uF" H 5900 3750 60  0000 L CNN
 F 2 "CAPC1608" H 5850 3900 60  0001 C CNN
@@
 $EndComp
 $Comp
-L C C?
+L C C30
 U 1 1 52414FE7
 P 8550 4100
-F 0 "C?" H 8600 4250 60  0000 L CNN
+F 0 "C30" H 8600 4250 60  0000 L CNN
 F 1 "0.01uF" H 8600 3950 60  0000 L CNN
 F 2 "CAPC1608" H 8550 4100 60  0001 C CNN
@@
 $EndComp
 $Comp
-L C C?
+L C C24
 U 1 1 52414FF2
 P 7150 3000
-F 0 "C?" H 7200 3150 60  0000 L CNN
+F 0 "C24" H 7200 3150 60  0000 L CNN
 F 1 "100pF" H 7200 2850 60  0000 L CNN
 F 2 "CAPC1608" H 7150 3000 60  0001 C CNN
@@
 $EndComp
 $Comp
-L C C?
+L C C26
 U 1 1 52414FFD
 P 10050 3300
-F 0 "C?" H 10100 3450 60  0000 L CNN
+F 0 "C26" H 10100 3450 60  0000 L CNN
 F 1 "100pF" H 10100 3150 60  0000 L CNN
 F 2 "CAPC1608" H 10050 3300 60  0001 C CNN
@@
 $EndComp
 $Comp
-L R R?
+L R R21
 U 1 1 52415008
 P 6450 3900
-F 0 "R?" H 6450 4000 50  0000 C CNN
+F 0 "R21" H 6450 4000 50  0000 C CNN
 F 1 "1k" H 6450 3900 50  0000 C CNN
 F 2 "RESC1608" H 6450 3900 60  0001 C CNN
@@
 $EndComp
 $Comp
-L R R?
+L R R22
 U 1 1 52415013
 P 9150 4100
-F 0 "R?" H 9150 4200 50  0000 C CNN
+F 0 "R22" H 9150 4200 50  0000 C CNN
 F 1 "1k" H 9150 4100 50  0000 C CNN
 F 2 "RESC1608" H 9150 4100 60  0001 C CNN
@@
 $EndComp
 $Comp
-L R R?
+L R R18
 U 1 1 5241501E
 P 7150 3400
-F 0 "R?" H 7150 3500 50  0000 C CNN
+F 0 "R18" H 7150 3500 50  0000 C CNN
 F 1 "10k" H 7150 3400 50  0000 C CNN
 F 2 "RESC1608" H 7150 3400 60  0001 C CNN
@@
 $EndComp
 $Comp
-L R R?
+L R R20
 U 1 1 52415029
 P 10050 3700
-F 0 "R?" H 10050 3800 50  0000 C CNN
+F 0 "R20" H 10050 3800 50  0000 C CNN
 F 1 "10k" H 10050 3700 50  0000 C CNN
 F 2 "RESC1608" H 10050 3700 60  0001 C CNN
@@
 $EndComp
 $Comp
-L C C?
+L C C25
 U 1 1 52415034
 P 7950 3000
-F 0 "C?" H 8000 3150 60  0000 L CNN
+F 0 "C25" H 8000 3150 60  0000 L CNN
 F 1 "0.1uF" H 8000 2850 60  0000 L CNN
 F 2 "CAPC1608" H 7950 3000 60  0001 C CNN

Commit message: Map test points
Parts:
- TP3, TP4: Distributor Part No (none) -> 5015KCT-ND; MFR Name (none) -> Keystone; MFR Part No (none) -> 5015
Changed lines of the file:
@@
 F 2 "" H 10700 3600 60  0000 C CNN
 F 3 "" H 10700 3600 60  0000 C CNN
+F 4 "Keystone" H 10700 3600 60  0001 C CNN "MFR Name"
+F 5 "5015" H 10700 3600 60  0001 C CNN "MFR Part No"
+F 6 "5015KCT-ND" H 10700 3600 60  0001 C CNN "Distributor Part No"
 	1    10700 3600
 	1    0    0    -1
@@
 F 2 "" H 900 3400 60  0000 C CNN
 F 3 "" H 900 3400 60  0000 C CNN
+F 4 "Keystone" H 900 3400 60  0001 C CNN "MFR Name"
+F 5 "5015" H 900 3400 60  0001 C CNN "MFR Part No"
+F 6 "5015KCT-ND" H 900 3400 60  0001 C CNN "Distributor Part No"
 	1    900  3400
 	1    0    0    -1

Commit message: Add power section. Switch to smaller pot
Connections:
- net labels added: +3.3V
- net labels removed: +5V
Changed lines of the file:
@@
 $Descr A4 11693 8268
 encoding utf-8
-Sheet 6 7
+Sheet 6 8
 Title "Solid State Cosmic Ray Detector"
 Date "24 sep 2013"
@@
 $EndComp
 $Comp
-L GND #PWR046
+L GND #PWR51
 U 1 1 52414ECB
 P 2400 4200
-F 0 "#PWR046" H 2400 4200 30  0001 C CNN
+F 0 "#PWR51" H 2400 4200 30  0001 C CNN
 F 1 "GND" H 2400 4130 30  0001 C CNN
 F 2 "" H 2400 4200 60  0000 C CNN
@@
 $EndComp
 $Comp
-L GND #PWR047
+L GND #PWR50
 U 1 1 52414ED1
 P 1800 4000
-F 0 "#PWR047" H 1800 4000 30  0001 C CNN
+F 0 "#PWR50" H 1800 4000 30  0001 C CNN
 F 1 "GND" H 1800 3930 30  0001 C CNN
 F 2 "" H 1800 4000 60  0000 C CNN
@@
 $EndComp
 $Comp
-L GND #PWR048
+L GND #PWR52
 U 1 1 52414ED7
 P 4300 4200
-F 0 "#PWR048" H 4300 4200 30  0001 C CNN
+F 0 "#PWR52" H 4300 4200 30  0001 C CNN
 F 1 "GND" H 4300 4130 30  0001 C CNN
 F 2 "" H 4300 4200 60  0000 C CNN
@@
 $EndComp
 $Comp
-L +5V #PWR049
-U 1 1 52414EF3
-P 2400 2500
-F 0 "#PWR049" H 2400 2590 20  0001 C CNN
-F 1 "+5V" H 2400 2590 30  0000 C CNN
-F 2 "" H 2400 2500 60  0000 C CNN
-F 3 "" H 2400 2500 60  0000 C CNN
-	1    2400 2500
-	1    0    0    -1
-$EndComp
-$Comp
 L C C22
 U 1 1 52414EFE
@@
 Connection ~ 1600 3000
 $Comp
-L GND #PWR050
+L GND #PWR47
 U 1 1 52414F45
 P 3100 2600
-F 0 "#PWR050" H 3100 2600 30  0001 C CNN
+F 0 "#PWR47" H 3100 2600 30  0001 C CNN
 F 1 "GND" H 3100 2530 30  0001 C CNN
 F 2 "" H 3100 2600 60  0000 C CNN
@@
 Connection ~ 7500 3400
 $Comp
-L GND #PWR051
+L GND #PWR49
 U 1 1 52414F68
 P 8300 3000
-F 0 "#PWR051" H 8300 3000 30  0001 C CNN
+F 0 "#PWR49" H 8300 3000 30  0001 C CNN
 F 1 "GND" H 8300 2930 30  0001 C CNN
 F 2 "" H 8300 3000 60  0000 C CNN
@@
 Wire Wire Line
 	8300 3000 8200 3000
-$Comp
-L +5V #PWR052
-U 1 1 52414F6F
-P 7600 2900
-F 0 "#PWR052" H 7600 2990 20  0001 C CNN
-F 1 "+5V" H 7600 2990 30  0000 C CNN
-F 2 "" H 7600 2900 60  0000 C CNN
-F 3 "" H 7600 2900 60  0000 C CNN
-	1    7600 2900
-	1    0    0    -1
-$EndComp
 Wire Wire Line
 	7600 2900 7600 3700
@@
 Connection ~ 10400 3700
 $Comp
-L GND #PWR053
+L GND #PWR55
 U 1 1 52414F87
 P 9500 4600
-F 0 "#PWR053" H 9500 4600 30  0001 C CNN
+F 0 "#PWR55" H 9500 4600 30  0001 C CNN
 F 1 "GND" H 9500 4530 30  0001 C CNN
 F 2 "" H 9500 4600 60  0000 C CNN
@@
 $EndComp
 $Comp
-L GND #PWR054
+L GND #PWR54
 U 1 1 52414F8D
 P 7600 4600
-F 0 "#PWR054" H 7600 4600 30  0001 C CNN
+F 0 "#PWR54" H 7600 4600 30  0001 C CNN
 F 1 "GND" H 7600 4530 30  0001 C CNN
 F 2 "" H 7600 4600 60  0000 C CNN
@@
 $EndComp
 $Comp
-L GND #PWR055
+L GND #PWR53
 U 1 1 52414F93
 P 7000 4400
-F 0 "#PWR055" H 7000 4400 30  0001 C CNN
+F 0 "#PWR53" H 7000 4400 30  0001 C CNN
 F 1 "GND" H 7000 4330 30  0001 C CNN
 F 2 "" H 7000 4400 60  0000 C CNN
@@
 	0    -1   -1   0
 $EndComp
+$Comp
+L +3.3V #PWR46
+U 1 1 5241F733
+P 2400 2500
+F 0 "#PWR46" H 2400 2460 30  0001 C CNN
+F 1 "+3.3V" H 2400 2610 30  0000 C CNN
+F 2 "" H 2400 2500 60  0000 C CNN
+F 3 "" H 2400 2500 60  0000 C CNN
+	1    2400 2500
+	1    0    0    -1
+$EndComp
+$Comp
+L +3.3V #PWR48
+U 1 1 5241F742
+P 7600 2900
+F 0 "#PWR48" H 7600 2860 30  0001 C CNN
+F 1 "+3.3V" H 7600 3010 30  0000 C CNN
+F 2 "" H 7600 2900 60  0000 C CNN
+F 3 "" H 7600 2900 60  0000 C CNN
+	1    7600 2900
+	1    0    0    -1
+$EndComp
 $EndSCHEMATC
