File: Hardware/Amp1.sch (KiCad schematic (older format))
At the start: 23 parts

Commit message: Initial annotation
Parts:
- gave numbers to parts that had none: 21
Changed lines of the file:
@@
 $EndDescr
 $Comp
-L OPAMP-DUAL U?
+L OPAMP-DUAL U1
 U 1 1 523CFEC7
 P 2400 3700
-F 0 "U?" H 2150 3800 50  0000 L CNN
+F 0 "U1" H 2150 3800 50  0000 L CNN
 F 1 "MAX4477" H 2150 3700 50  0000 L CNN
 F 2 "" H 2400 3700 60  0000 C CNN
@@
 $EndComp
 $Comp
-L GND #PWR?
+L GND #PWR16
 U 1 1 523CFED3
 P 2400 4200
-F 0 "#PWR?" H 2400 4200 30  0001 C CNN
+F 0 "#PWR16" H 2400 4200 30  0001 C CNN
 F 1 "GND" H 2400 4130 30  0001 C CNN
 F 2 "" H 2400 4200 60  0000 C CNN
@@
 $EndComp
 $Comp
-L GND #PWR?
+L GND #PWR15
 U 1 1 523CFED9
 P 1800 4000
-F 0 "#PWR?" H 1800 4000 30  0001 C CNN
+F 0 "#PWR15" H 1800 4000 30  0001 C CNN
 F 1 "GND" H 1800 3930 30  0001 C CNN
 F 2 "" H 1800 4000 60  0000 C CNN
@@
 $EndComp
 $Comp
-L GND #PWR?
+L GND #PWR17
 U 1 1 523CFEDF
 P 4300 4200
-F 0 "#PWR?" H 4300 4200 30  0001 C CNN
+F 0 "#PWR17" H 4300 4200 30  0001 C CNN
 F 1 "GND" H 4300 4130 30  0001 C CNN
 F 2 "" H 4300 4200 60  0000 C CNN
@@
 $EndComp
 $Comp
-L R R?
+L R R3
 U 1 1 523CFEE7
 P 1950 3000
-F 0 "R?" H 1950 3100 50  0000 C CNN
+F 0 "R3" H 1950 3100 50  0000 C CNN
 F 1 "10M" H 1950 3000 50  0000 C CNN
 F 2 "RESC1608" H 1950 3000 60  0001 C CNN
@@
 $EndComp
 $Comp
-L C C?
+L C C2
 U 1 1 523CFEEF
 P 1950 2600
-F 0 "C?" H 2000 2750 60  0000 L CNN
+F 0 "C2" H 2000 2750 60  0000 L CNN
 F 1 "4.7pF" H 2000 2450 60  0000 L CNN
 F 2 "CAPC1608" H 1950 2600 60  0001 C CNN
@@
 $EndComp
 $Comp
-L +5V #PWR?
+L +5V #PWR11
 U 1 1 523CFEF5
 P 2400 2500
-F 0 "#PWR?" H 2400 2590 20  0001 C CNN
+F 0 "#PWR11" H 2400 2590 20  0001 C CNN
 F 1 "+5V" H 2400 2590 30  0000 C CNN
 F 2 "" H 2400 2500 60  0000 C CNN
@@
 $EndComp
 $Comp
-L C C?
+L C C3
 U 1 1 523CFEFD
 P 2750 2600
-F 0 "C?" H 2800 2750 60  0000 L CNN
+F 0 "C3" H 2800 2750 60  0000 L CNN
 F 1 "0.1uF" H 2800 2450 60  0000 L CNN
 F 2 "CAPC1608" H 2750 2600 60  0001 C CNN
@@
 $EndComp
 $Comp
-L R R?
+L R R6
 U 1 1 523CFF0D
 P 3950 3700
-F 0 "R?" H 3950 3800 50  0000 C CNN
+F 0 "R6" H 3950 3800 50  0000 C CNN
 F 1 "1k" H 3950 3700 50  0000 C CNN
 F 2 "RESC1608" H 3950 3700 60  0001 C CNN
@@
 $EndComp
 $Comp
-L R R?
+L R R4
 U 1 1 523CFF15
 P 4850 3300
-F 0 "R?" H 4850 3400 50  0000 C CNN
+F 0 "R4" H 4850 3400 50  0000 C CNN
 F 1 "10k" H 4850 3300 50  0000 C CNN
 F 2 "RESC1608" H 4850 3300 60  0001 C CNN
@@
 $EndComp
 $Comp
-L C C?
+L C C4
 U 1 1 523CFF1D
 P 4850 2900
-F 0 "C?" H 4900 3050 60  0000 L CNN
+F 0 "C4" H 4900 3050 60  0000 L CNN
 F 1 "100pF" H 4900 2750 60  0000 L CNN
 F 2 "CAPC1608" H 4850 2900 60  0001 C CNN
@@
 Connection ~ 1600 3000
 $Comp
-L GND #PWR?
+L GND #PWR12
 U 1 1 523CFF43
 P 3100 2600
-F 0 "#PWR?" H 3100 2600 30  0001 C CNN
+F 0 "#PWR12" H 3100 2600 30  0001 C CNN
 F 1 "GND" H 3100 2530 30  0001 C CNN
 F 2 "" H 3100 2600 60  0000 C CNN
@@
 Connection ~ 2400 2600
 $Comp
-L C C?
+L C C8
 U 1 1 523CFF56
 P 1250 3500
-F 0 "C?" H 1300 3650 60  0000 L CNN
+F 0 "C8" H 1300 3650 60  0000 L CNN
 F 1 "0.01uF" H 1300 3350 60  0000 L CNN
 F 2 "CAPC1608" H 1250 3500 60  0001 C CNN
@@
 Connection ~ 7500 3400
 $Comp
-L GND #PWR?
+L GND #PWR14
 U 1 1 523CFF91
 P 8300 3000
-F 0 "#PWR?" H 8300 3000 30  0001 C CNN
+F 0 "#PWR14" H 8300 3000 30  0001 C CNN
 F 1 "GND" H 8300 2930 30  0001 C CNN
 F 2 "" H 8300 3000 60  0000 C CNN
@@
 	8300 3000 8200 3000
 $Comp
-L +5V #PWR?
+L +5V #PWR13
 U 1 1 523CFF98
 P 7600 2900
-F 0 "#PWR?" H 7600 2990 20  0001 C CNN
+F 0 "#PWR13" H 7600 2990 20  0001 C CNN
 F 1 "+5V" H 7600 2990 30  0000 C CNN
 F 2 "" H 7600 2900 60  0000 C CNN
@@
 Connection ~ 10400 3700
 $Comp
-L GND #PWR?
+L GND #PWR20
 U 1 1 523CFFD6
 P 9500 4600
-F 0 "#PWR?" H 9500 4600 30  0001 C CNN
+F 0 "#PWR20" H 9500 4600 30  0001 C CNN
 F 1 "GND" H 9500 4530 30  0001 C CNN
 F 2 "" H 9500 4600 60  0000 C CNN
@@
 $EndComp
 $Comp
-L GND #PWR?
+L GND #PWR19
 U 1 1 523CFFDC
 P 7600 4600
-F 0 "#PWR?" H 7600 4600 30  0001 C CNN
+F 0 "#PWR19" H 7600 4600 30  0001 C CNN
 F 1 "GND" H 7600 4530 30  0001 C CNN
 F 2 "" H 7600 4600 60  0000 C CNN
@@
 $EndComp
 $Comp
-L GND #PWR?
+L GND #PWR18
 U 1 1 523CFFE2
 P 7000 4400
-F 0 "#PWR?" H 7000 4400 30  0001 C CNN
+F 0 "#PWR18" H 7000 4400 30  0001 C CNN
 F 1 "GND" H 7000 4330 30  0001 C CNN
 F 2 "" H 7000 4400 60  0000 C CNN
@@
 Connection ~ 10700 4300
 $Comp
-L TP TP?
+L TP TP2
 U 1 1 523CFFF1
 P 10700 3600
-F 0 "TP?" H 10700 3950 60  0000 C CNN
+F 0 "TP2" H 10700 3950 60  0000 C CNN
 F 1 "Out1" H 10700 3850 60  0000 C CNN
 F 2 "" H 10700 3600 60  0000 C CNN
@@
 Connection ~ 10700 3700
 $Comp
-L TP TP?
+L TP TP1
 U 1 1 523CFFF8
 P 900 3400
-F 0 "TP?" H 900 3750 60  0000 C CNN
+F 0 "TP1" H 900 3750 60  0000 C CNN
 F 1 "In1" H 900 3650 60  0000 C CNN
 F 2 "" H 900 3400 60  0000 C CNN
@@
 In
 $Comp
-L OPAMP-DUAL U?
+L OPAMP-DUAL U1
 U 2 1 523FC6E8
 P 4900 3900
-F 0 "U?" H 4650 4000 50  0000 L CNN
+F 0 "U1" H 4650 4000 50  0000 L CNN
 F 1 "MAX4477" H 4650 3900 50  0000 L CNN
 F 2 "" H 4900 3900 60  0000 C CNN
@@
 $EndComp
 $Comp
-L OPAMP-DUAL U?
+L OPAMP-DUAL U2
 U 1 1 523FC6F1
 P 7600 4100
-F 0 "U?" H 7350 4200 50  0000 L CNN
+F 0 "U2" H 7350 4200 50  0000 L CNN
 F 1 "MAX4477" H 7350 4100 50  0000 L CNN
 F 2 "" H 7600 4100 60  0000 C CNN
@@
 $EndComp
 $Comp
-L OPAMP-DUAL U?
+L OPAMP-DUAL U2
 U 2 1 523FC6FA
 P 10100 4300
-F 0 "U?" H 9850 4400 50  0000 L CNN
+F 0 "U2" H 9850 4400 50  0000 L CNN
 F 1 "MAX4477" H 9850 4300 50  0000 L CNN
 F 2 "" H 10100 4300 60  0000 C CNN
@@
 $EndComp
 $Comp
-L C C?
+L C C9
 U 1 1 524124C8
 P 3350 3700
-F 0 "C?" H 3400 3850 60  0000 L CNN
+F 0 "C9" H 3400 3850 60  0000 L CNN
 F 1 "0.01uF" H 3400 3550 60  0000 L CNN
 F 2 "CAPC1608" H 3350 3700 60  0001 C CNN
@@
 $EndComp
 $Comp
-L C C?
+L C C10
 U 1 1 524124D3
 P 5850 3900
-F 0 "C?" H 5900 4050 60  0000 L CNN
+F 0 "C10" H 5900 4050 60  0000 L CNN
 F 1 "0.01uF" H 5900 3750 60  0000 L CNN
 F 2 "CAPC1608" H 5850 3900 60  0001 C CNN
@@
 $EndComp
 $Comp
-L C C?
+L C C11
 U 1 1 524124DE
 P 8550 4100
-F 0 "C?" H 8600 4250 60  0000 L CNN
+F 0 "C11" H 8600 4250 60  0000 L CNN
 F 1 "0.01uF" H 8600 3950 60  0000 L CNN
 F 2 "CAPC1608" H 8550 4100 60  0001 C CNN
@@
 $EndComp
 $Comp
-L C C?
+L C C5
 U 1 1 5241258A
 P 7150 3000
-F 0 "C?" H 7200 3150 60  0000 L CNN
+F 0 "C5" H 7200 3150 60  0000 L CNN
 F 1 "100pF" H 7200 2850 60  0000 L CNN
 F 2 "CAPC1608" H 7150 3000 60  0001 C CNN
@@
 $EndComp
 $Comp
-L C C?
+L C C7
 U 1 1 52412595
 P 10050 3300
-F 0 "C?" H 10100 3450 60  0000 L CNN
+F 0 "C7" H 10100 3450 60  0000 L CNN
 F 1 "100pF" H 10100 3150 60  0000 L CNN
 F 2 "CAPC1608" H 10050 3300 60  0001 C CNN
@@
 $EndComp
 $Comp
-L R R?
+L R R8
 U 1 1 5241267F
 P 6450 3900
-F 0 "R?" H 6450 4000 50  0000 C CNN
+F 0 "R8" H 6450 4000 50  0000 C CNN
 F 1 "1k" H 6450 3900 50  0000 C CNN
 F 2 "RESC1608" H 6450 3900 60  0001 C CNN
@@
 $EndComp
 $Comp
-L R R?
+L R R9
 U 1 1 5241268A
 P 9150 4100
-F 0 "R?" H 9150 4200 50  0000 C CNN
+F 0 "R9" H 9150 4200 50  0000 C CNN
 F 1 "1k" H 9150 4100 50  0000 C CNN
 F 2 "RESC1608" H 9150 4100 60  0001 C CNN
@@
 $EndComp
 $Comp
-L R R?
+L R R5
 U 1 1 52412715
 P 7150 3400
-F 0 "R?" H 7150 3500 50  0000 C CNN
+F 0 "R5" H 7150 3500 50  0000 C CNN
 F 1 "10k" H 7150 3400 50  0000 C CNN
 F 2 "RESC1608" H 7150 3400 60  0001 C CNN
@@
 $EndComp
 $Comp
-L R R?
+L R R7
 U 1 1 52412720
 P 10050 3700
-F 0 "R?" H 10050 3800 50  0000 C CNN
+F 0 "R7" H 10050 3800 50  0000 C CNN
 F 1 "10k" H 10050 3700 50  0000 C CNN
 F 2 "RESC1608" H 10050 3700 60  0001 C CNN
@@
 $EndComp
 $Comp
-L C C?
+L C C6
 U 1 1 52412801
 P 7950 3000
-F 0 "C?" H 8000 3150 60  0000 L CNN
+F 0 "C6" H 8000 3150 60  0000 L CNN
 F 1 "0.1uF" H 8000 2850 60  0000 L CNN
 F 2 "CAPC1608" H 7950 3000 60  0001 C CNN

Commit message: Map test points
Parts:
- TP1, TP2: Distributor Part No (none) -> 5015KCT-ND; MFR Name (none) -> Keystone; MFR Part No (none) -> 5015
Changed lines of the file:
@@
 F 2 "" H 10700 3600 60  0000 C CNN
 F 3 "" H 10700 3600 60  0000 C CNN
+F 4 "Keystone" H 10700 3600 60  0001 C CNN "MFR Name"
+F 5 "5015" H 10700 3600 60  0001 C CNN "MFR Part No"
+F 6 "5015KCT-ND" H 10700 3600 60  0001 C CNN "Distributor Part No"
 	1    10700 3600
 	1    0    0    -1
@@
 F 2 "" H 900 3400 60  0000 C CNN
 F 3 "" H 900 3400 60  0000 C CNN
+F 4 "Keystone" H 900 3400 60  0001 C CNN "MFR Name"
+F 5 "5015" H 900 3400 60  0001 C CNN "MFR Part No"
+F 6 "5015KCT-ND" H 900 3400 60  0001 C CNN "Distributor Part No"
 	1    900  3400
 	1    0    0    -1

Commit message: Add power section. Switch to smaller pot
Connections:
- net labels added: +3.3V
- net labels removed: +5V
Changed lines of the file:
@@
 $Descr A4 11693 8268
 encoding utf-8
-Sheet 3 7
+Sheet 3 8
 Title "Solid State Cosmic Ray Detector"
 Date "24 sep 2013"
@@
 $EndComp
 $Comp
-L GND #PWR011
+L GND #PWR16
 U 1 1 523CFED3
 P 2400 4200
-F 0 "#PWR011" H 2400 4200 30  0001 C CNN
+F 0 "#PWR16" H 2400 4200 30  0001 C CNN
 F 1 "GND" H 2400 4130 30  0001 C CNN
 F 2 "" H 2400 4200 60  0000 C CNN
@@
 $EndComp
 $Comp
-L GND #PWR012
+L GND #PWR15
 U 1 1 523CFED9
 P 1800 4000
-F 0 "#PWR012" H 1800 4000 30  0001 C CNN
+F 0 "#PWR15" H 1800 4000 30  0001 C CNN
 F 1 "GND" H 1800 3930 30  0001 C CNN
 F 2 "" H 1800 4000 60  0000 C CNN
@@
 $EndComp
 $Comp
-L GND #PWR013
+L GND #PWR17
 U 1 1 523CFEDF
 P 4300 4200
-F 0 "#PWR013" H 4300 4200 30  0001 C CNN
+F 0 "#PWR17" H 4300 4200 30  0001 C CNN
 F 1 "GND" H 4300 4130 30  0001 C CNN
 F 2 "" H 4300 4200 60  0000 C CNN
@@
 $EndComp
 $Comp
-L +5V #PWR014
-U 1 1 523CFEF5
-P 2400 2500
-F 0 "#PWR014" H 2400 2590 20  0001 C CNN
-F 1 "+5V" H 2400 2590 30  0000 C CNN
-F 2 "" H 2400 2500 60  0000 C CNN
-F 3 "" H 2400 2500 60  0000 C CNN
-	1    2400 2500
-	1    0    0    -1
-$EndComp
-$Comp
 L C C3
 U 1 1 523CFEFD
@@
 Connection ~ 1600 3000
 $Comp
-L GND #PWR015
+L GND #PWR12
 U 1 1 523CFF43
 P 3100 2600
-F 0 "#PWR015" H 3100 2600 30  0001 C CNN
+F 0 "#PWR12" H 3100 2600 30  0001 C CNN
 F 1 "GND" H 3100 2530 30  0001 C CNN
 F 2 "" H 3100 2600 60  0000 C CNN
@@
 Connection ~ 7500 3400
 $Comp
-L GND #PWR016
+L GND #PWR14
 U 1 1 523CFF91
 P 8300 3000
-F 0 "#PWR016" H 8300 3000 30  0001 C CNN
+F 0 "#PWR14" H 8300 3000 30  0001 C CNN
 F 1 "GND" H 8300 2930 30  0001 C CNN
 F 2 "" H 8300 3000 60  0000 C CNN
@@
 Wire Wire Line
 	8300 3000 8200 3000
-$Comp
-L +5V #PWR017
-U 1 1 523CFF98
-P 7600 2900
-F 0 "#PWR017" H 7600 2990 20  0001 C CNN
-F 1 "+5V" H 7600 2990 30  0000 C CNN
-F 2 "" H 7600 2900 60  0000 C CNN
-F 3 "" H 7600 2900 60  0000 C CNN
-	1    7600 2900
-	1    0    0    -1
-$EndComp
 Wire Wire Line
 	7600 2900 7600 3700
@@
 Connection ~ 10400 3700
 $Comp
-L GND #PWR018
+L GND #PWR20
 U 1 1 523CFFD6
 P 9500 4600
-F 0 "#PWR018" H 9500 4600 30  0001 C CNN
+F 0 "#PWR20" H 9500 4600 30  0001 C CNN
 F 1 "GND" H 9500 4530 30  0001 C CNN
 F 2 "" H 9500 4600 60  0000 C CNN
@@
 $EndComp
 $Comp
-L GND #PWR019
+L GND #PWR19
 U 1 1 523CFFDC
 P 7600 4600
-F 0 "#PWR019" H 7600 4600 30  0001 C CNN
+F 0 "#PWR19" H 7600 4600 30  0001 C CNN
 F 1 "GND" H 7600 4530 30  0001 C CNN
 F 2 "" H 7600 4600 60  0000 C CNN
@@
 $EndComp
 $Comp
-L GND #PWR020
+L GND #PWR18
 U 1 1 523CFFE2
 P 7000 4400
-F 0 "#PWR020" H 7000 4400 30  0001 C CNN
+F 0 "#PWR18" H 7000 4400 30  0001 C CNN
 F 1 "GND" H 7000 4330 30  0001 C CNN
 F 2 "" H 7000 4400 60  0000 C CNN
@@
 	0    -1   -1   0
 $EndComp
+$Comp
+L +3.3V #PWR11
+U 1 1 5241F6B5
+P 2400 2500
+F 0 "#PWR11" H 2400 2460 30  0001 C CNN
+F 1 "+3.3V" H 2400 2610 30  0000 C CNN
+F 2 "" H 2400 2500 60  0000 C CNN
+F 3 "" H 2400 2500 60  0000 C CNN
+	1    2400 2500
+	1    0    0    -1
+$EndComp
+$Comp
+L +3.3V #PWR13
+U 1 1 5241F6C4
+P 7600 2900
+F 0 "#PWR13" H 7600 2860 30  0001 C CNN
+F 1 "+3.3V" H 7600 3010 30  0000 C CNN
+F 2 "" H 7600 2900 60  0000 C CNN
+F 3 "" H 7600 2900 60  0000 C CNN
+	1    7600 2900
+	1    0    0    -1
+$EndComp
 $EndSCHEMATC
