File: Hardware/Det2.sch (KiCad schematic (older format))
At the start: 11 parts

Commit message: Initial annotation
Parts:
- gave numbers to parts that had none: 11
Changed lines of the file:
@@
 $EndDescr
 $Comp
-L GND #PWR?
+L GND #PWR58
 U 1 1 524151B0
 P 2700 3600
-F 0 "#PWR?" H 2700 3600 30  0001 C CNN
+F 0 "#PWR58" H 2700 3600 30  0001 C CNN
 F 1 "GND" H 2700 3530 30  0001 C CNN
 F 2 "" H 2700 3600 60  0000 C CNN
@@
 $EndComp
 $Comp
-L GND #PWR?
+L GND #PWR59
 U 1 1 524151B6
 P 3100 3600
-F 0 "#PWR?" H 3100 3600 30  0001 C CNN
+F 0 "#PWR59" H 3100 3600 30  0001 C CNN
 F 1 "GND" H 3100 3530 30  0001 C CNN
 F 2 "" H 3100 3600 60  0000 C CNN
@@
 $EndComp
 $Comp
-L GND #PWR?
+L GND #PWR61
 U 1 1 524151BC
 P 3900 3600
-F 0 "#PWR?" H 3900 3600 30  0001 C CNN
+F 0 "#PWR61" H 3900 3600 30  0001 C CNN
 F 1 "GND" H 3900 3530 30  0001 C CNN
 F 2 "" H 3900 3600 60  0000 C CNN
@@
 $EndComp
 $Comp
-L GND #PWR?
+L GND #PWR60
 U 1 1 524151C2
 P 3500 3600
-F 0 "#PWR?" H 3500 3600 30  0001 C CNN
+F 0 "#PWR60" H 3500 3600 30  0001 C CNN
 F 1 "GND" H 3500 3530 30  0001 C CNN
 F 2 "" H 3500 3600 60  0000 C CNN
@@
 Out
 $Comp
-L +12V #PWR?
+L +12V #PWR56
 U 1 1 524151CD
 P 2000 2200
-F 0 "#PWR?" H 2000 2150 20  0001 C CNN
+F 0 "#PWR56" H 2000 2150 20  0001 C CNN
 F 1 "+12V" H 2000 2300 30  0000 C CNN
 F 2 "" H 2000 2200 60  0000 C CNN
@@
 $EndComp
 $Comp
-L R R?
+L R R23
 U 1 1 524151D8
 P 2000 2550
-F 0 "R?" H 2000 2650 50  0000 C CNN
+F 0 "R23" H 2000 2650 50  0000 C CNN
 F 1 "1M" H 2000 2550 50  0000 C CNN
 F 2 "RESC1608" H 2000 2550 60  0001 C CNN
@@
 $EndComp
 $Comp
-L GND #PWR?
+L GND #PWR57
 U 1 1 524151DE
 P 2000 3600
-F 0 "#PWR?" H 2000 3600 30  0001 C CNN
+F 0 "#PWR57" H 2000 3600 30  0001 C CNN
 F 1 "GND" H 2000 3530 30  0001 C CNN
 F 2 "" H 2000 3600 60  0000 C CNN
@@
 Connection ~ 2000 2900
 $Comp
-L DIODE-PHOTO D?
+L DIODE-PHOTO D16
 U 1 1 524151EC
 P 5500 3250
-F 0 "D?" H 5500 3350 60  0000 C CNN
+F 0 "D16" H 5500 3350 60  0000 C CNN
 F 1 "VBPW34FASR" H 5500 3150 60  0000 C CNN
 F 2 "DIOC-BPW34R" H 5500 3250 60  0001 C CNN
@@
 $EndComp
 $Comp
-L GND #PWR?
+L GND #PWR62
 U 1 1 524151F2
 P 4300 3600
-F 0 "#PWR?" H 4300 3600 30  0001 C CNN
+F 0 "#PWR62" H 4300 3600 30  0001 C CNN
 F 1 "GND" H 4300 3530 30  0001 C CNN
 F 2 "" H 4300 3600 60  0000 C CNN
@@
 $EndComp
 $Comp
-L GND #PWR?
+L GND #PWR63
 U 1 1 524151F8
 P 4700 3600
-F 0 "#PWR?" H 4700 3600 30  0001 C CNN
+F 0 "#PWR63" H 4700 3600 30  0001 C CNN
 F 1 "GND" H 4700 3530 30  0001 C CNN
 F 2 "" H 4700 3600 60  0000 C CNN
@@
 $EndComp
 $Comp
-L GND #PWR?
+L GND #PWR65
 U 1 1 524151FE
 P 5500 3600
-F 0 "#PWR?" H 5500 3600 30  0001 C CNN
+F 0 "#PWR65" H 5500 3600 30  0001 C CNN
 F 1 "GND" H 5500 3530 30  0001 C CNN
 F 2 "" H 5500 3600 60  0000 C CNN
@@
 $EndComp
 $Comp
-L GND #PWR?
+L GND #PWR64
 U 1 1 52415204
 P 5100 3600
-F 0 "#PWR?" H 5100 3600 30  0001 C CNN
+F 0 "#PWR64" H 5100 3600 30  0001 C CNN
 F 1 "GND" H 5100 3530 30  0001 C CNN
 F 2 "" H 5100 3600 60  0000 C CNN
@@
 Connection ~ 5500 2900
 $Comp
-L DIODE-PHOTO D?
+L DIODE-PHOTO D15
 U 1 1 52415222
 P 5100 3250
-F 0 "D?" H 5100 3350 60  0000 C CNN
+F 0 "D15" H 5100 3350 60  0000 C CNN
 F 1 "VBPW34FASR" H 5100 3150 60  0000 C CNN
 F 2 "DIOC-BPW34R" H 5100 3250 60  0001 C CNN
@@
 $EndComp
 $Comp
-L DIODE-PHOTO D?
+L DIODE-PHOTO D14
 U 1 1 5241522B
 P 4700 3250
-F 0 "D?" H 4700 3350 60  0000 C CNN
+F 0 "D14" H 4700 3350 60  0000 C CNN
 F 1 "VBPW34FASR" H 4700 3150 60  0000 C CNN
 F 2 "DIOC-BPW34R" H 4700 3250 60  0001 C CNN
@@
 $EndComp
 $Comp
-L DIODE-PHOTO D?
+L DIODE-PHOTO D13
 U 1 1 52415234
 P 4300 3250
-F 0 "D?" H 4300 3350 60  0000 C CNN
+F 0 "D13" H 4300 3350 60  0000 C CNN
 F 1 "VBPW34FASR" H 4300 3150 60  0000 C CNN
 F 2 "DIOC-BPW34R" H 4300 3250 60  0001 C CNN
@@
 $EndComp
 $Comp
-L DIODE-PHOTO D?
+L DIODE-PHOTO D12
 U 1 1 5241523D
 P 3900 3250
-F 0 "D?" H 3900 3350 60  0000 C CNN
+F 0 "D12" H 3900 3350 60  0000 C CNN
 F 1 "VBPW34FASR" H 3900 3150 60  0000 C CNN
 F 2 "DIOC-BPW34R" H 3900 3250 60  0001 C CNN
@@
 $EndComp
 $Comp
-L DIODE-PHOTO D?
+L DIODE-PHOTO D11
 U 1 1 52415246
 P 3500 3250
-F 0 "D?" H 3500 3350 60  0000 C CNN
+F 0 "D11" H 3500 3350 60  0000 C CNN
 F 1 "VBPW34FASR" H 3500 3150 60  0000 C CNN
 F 2 "DIOC-BPW34R" H 3500 3250 60  0001 C CNN
@@
 $EndComp
 $Comp
-L DIODE-PHOTO D?
+L DIODE-PHOTO D10
 U 1 1 5241524F
 P 3100 3250
-F 0 "D?" H 3100 3350 60  0000 C CNN
+F 0 "D10" H 3100 3350 60  0000 C CNN
 F 1 "VBPW34FASR" H 3100 3150 60  0000 C CNN
 F 2 "DIOC-BPW34R" H 3100 3250 60  0001 C CNN
@@
 $EndComp
 $Comp
-L DIODE-PHOTO D?
+L DIODE-PHOTO D9
 U 1 1 52415258
 P 2700 3250
-F 0 "D?" H 2700 3350 60  0000 C CNN
+F 0 "D9" H 2700 3350 60  0000 C CNN
 F 1 "VBPW34FASR" H 2700 3150 60  0000 C CNN
 F 2 "DIOC-BPW34R" H 2700 3250 60  0001 C CNN
@@
 $EndComp
 $Comp
-L R R?
+L R R24
 U 1 1 52415263
 P 2350 2900
-F 0 "R?" H 2350 3000 50  0000 C CNN
+F 0 "R24" H 2350 3000 50  0000 C CNN
 F 1 "10M" H 2350 2900 50  0000 C CNN
 F 2 "RESC1608" H 2350 2900 60  0001 C CNN
@@
 $EndComp
 $Comp
-L C C?
+L C C31
 U 1 1 5241526E
 P 2000 3250
-F 0 "C?" H 2050 3400 60  0000 L CNN
+F 0 "C31" H 2050 3400 60  0000 L CNN
 F 1 "0.1uF" H 2050 3100 60  0000 L CNN
 F 2 "CAPC1608" H 2000 3250 60  0001 C CNN
